File: Antenna-Array-Switch-PCB/Microcontroller.kicad_sch (KiCad schematic)
At the start: 0 parts

Commit message: PCB: Add MCU, switch
Parts:
- added D10, D7, D8, D9: LED, symbol Device:LED
- added R13, R14, R15, R16, R17, R18, R19, R21, R23: 10k, symbol Device:R
- added R20, R22, R24: 12k, symbol Device:R
- added SW1, SW2: SW_Push, symbol Switch:SW_Push
- added U9: RP2040-Zero, 00-project-footprints:RP2040 Zero, symbol 00-project-symbols:RP2040-Zero
Connections:
- new net: D7.1 (K), R14.1
- new net: D10.1 (K), R16.1
- new net: D8.1 (K), R13.1
- new net: D9.1 (K), R15.1
- new net +5V: U9.1 (5V)
- new net GNDA: R20.2, R22.2, R24.2
- new net GNDD: R13.2, R14.2, R15.2, R16.2, R17.2, R18.2, U9.2 (GND)
- new net GP_BUTTON_1: R17.1, SW1.1, U9.8 (GP15)
- new net GP_BUTTON_2: R18.1, SW2.1, U9.9 (GP14)
- new net LNA_ENABLE_0: U9.10 (GP0)
- new net LNA_ENABLE_1: U9.11 (GP1)
- new net LNA_ENABLE_2: U9.12 (GP2)
- new net LNA_ENABLE_3: U9.13 (GP3)
- new net LNA_ENABLE_4: U9.14 (GP4)
- new net LNA_ENABLE_5: U9.15 (GP5)
- new net LNA_ENABLE_6: U9.16 (GP6)
- new net LNA_ENABLE_7: U9.17 (GP7)
- new net MCU_3V3: SW1.2, SW2.2, U9.3 (3V3)
- new net STATUS_LED: D10.2 (A), U9.7 (GP26)
- new net SWITCH_CTRL1_AT_1V8: R19.2, R20.1
- new net SWITCH_CTRL1_AT_3V3: D7.2 (A), R19.1, U9.6 (GP27)
- new net SWITCH_CTRL2_AT_1V8: R21.2, R22.1
- new net SWITCH_CTRL2_AT_3V3: D8.2 (A), R21.1, U9.5 (GP28)
- new net SWITCH_CTRL3_AT_1V8: R23.2, R24.1
- new net SWITCH_CTRL3_AT_3V3: D9.2 (A), R23.1, U9.4 (GP29)
- no-connect marks 0 -> 6
Other:
- note added: "3V3 at GPIO -> 1V8 at Switch. Use voltage dividers. 3.3 × 12 / (10 + 12) = 1V8"

Commit message: PCB: Assign footprints
Parts:
- D10, D7, D8, D9: footprint (none) -> LED_SMD:LED_0603_1608Metric_Pad1.05x0.95mm_HandSolder
- R13, R14, R15, R16, R17, R18, R19, R20, R21, R22, R23, R24: footprint (none) -> Resistor_SMD:R_0603_1608Metric_Pad0.98x0.95mm_HandSolder
Changed lines of the file:
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@@
 			)
 		)
-		(property "Footprint" ""
+		(property "Footprint" "Resistor_SMD:R_0603_1608Metric_Pad0.98x0.95mm_HandSolder"
 			(at 156.972 67.31 90)
 			(hide yes)
@@
 			)
 		)
-		(property "Footprint" ""
+		(property "Footprint" "Resistor_SMD:R_0603_1608Metric_Pad0.98x0.95mm_HandSolder"
 			(at 134.112 151.13 90)
 			(hide yes)
@@
 			)
 		)
-		(property "Footprint" ""
+		(property "Footprint" "Resistor_SMD:R_0603_1608Metric_Pad0.98x0.95mm_HandSolder"
 			(at 184.912 55.88 90)
 			(hide yes)
@@
 			)
 		)
-		(property "Footprint" ""
+		(property "Footprint" "Resistor_SMD:R_0603_1608Metric_Pad0.98x0.95mm_HandSolder"
 			(at 212.852 55.88 90)
 			(hide yes)
@@
 			)
 		)
-		(property "Footprint" ""
+		(property "Footprint" "Resistor_SMD:R_0603_1608Metric_Pad0.98x0.95mm_HandSolder"
 			(at 231.648 148.59 90)
 			(hide yes)
@@
 			)
 		)
-		(property "Footprint" ""
+		(property "Footprint" "LED_SMD:LED_0603_1608Metric_Pad1.05x0.95mm_HandSolder"
 			(at 229.87 137.16 0)
 			(hide yes)
@@
 			)
 		)
-		(property "Footprint" ""
+		(property "Footprint" "LED_SMD:LED_0603_1608Metric_Pad1.05x0.95mm_HandSolder"
 			(at 99.06 134.62 0)
 			(hide yes)
@@
 			)
 		)
-		(property "Footprint" ""
+		(property "Footprint" "Resistor_SMD:R_0603_1608Metric_Pad0.98x0.95mm_HandSolder"
 			(at 240.538 148.59 90)
 			(hide yes)
@@
 			)
 		)
-		(property "Footprint" ""
+		(property "Footprint" "LED_SMD:LED_0603_1608Metric_Pad1.05x0.95mm_HandSolder"
 			(at 247.65 137.16 0)
 			(hide yes)
@@
 			)
 		)
-		(property "Footprint" ""
+		(property "Footprint" "Resistor_SMD:R_0603_1608Metric_Pad0.98x0.95mm_HandSolder"
 			(at 100.838 146.05 90)
 			(hide yes)
@@
 			)
 		)
-		(property "Footprint" ""
+		(property "Footprint" "LED_SMD:LED_0603_1608Metric_Pad1.05x0.95mm_HandSolder"
 			(at 238.76 137.16 0)
 			(hide yes)
@@
 			)
 		)
-		(property "Footprint" ""
+		(property "Footprint" "Resistor_SMD:R_0603_1608Metric_Pad0.98x0.95mm_HandSolder"
 			(at 184.912 67.31 90)
 			(hide yes)
@@
 			)
 		)
-		(property "Footprint" ""
+		(property "Footprint" "Resistor_SMD:R_0603_1608Metric_Pad0.98x0.95mm_HandSolder"
 			(at 249.428 148.59 90)
 			(hide yes)
@@
 			)
 		)
-		(property "Footprint" ""
+		(property "Footprint" "Resistor_SMD:R_0603_1608Metric_Pad0.98x0.95mm_HandSolder"
 			(at 156.972 55.88 90)
 			(hide yes)
@@
 			)
 		)
-		(property "Footprint" ""
+		(property "Footprint" "Resistor_SMD:R_0603_1608Metric_Pad0.98x0.95mm_HandSolder"
 			(at 212.852 67.31 90)
 			(hide yes)
@@
 			)
 		)
-		(property "Footprint" ""
+		(property "Footprint" "Resistor_SMD:R_0603_1608Metric_Pad0.98x0.95mm_HandSolder"
 			(at 146.558 151.13 90)
 			(hide yes)

Commit message: PCB: Finish footprint assignments
Parts:
- removed SW1, SW2: SW_Push, symbol Switch:SW_Push
- added SW1, SW2: TS-1187A-B-A-B, 00-lcsc-footprints:C318884_SW-SMD_4P-L5_1-W5_1-P3_70-LS6_5-TL_H1_5, symbol 00-lcsc-symbols:TS-1187A-B-A-B
Connections:
- net GP_BUTTON_1: now also SW1.3 (C), SW1.4 (D)
- net GP_BUTTON_2: now also SW2.3 (C), SW2.4 (D)
- net MCU_3V3: now also SW1.1 (A), SW1.2 (B), SW2.1 (A), SW2.2 (B)

Commit message: PCB, Docs: Layout, stackup, shielding
Parts:
- added J12: RFShield_OnePiece, RF_Shielding:Wuerth_36103305_30x30mm, symbol Device:RFShield_OnePiece
Connections:
- net GNDD is gone; now on net GNDA: R13.2, R14.2, R15.2, R16.2, R17.2, R18.2, U9.2 (GND)
- net GNDA: now also J12.1 (Shield)
Changed lines of the file:
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@@
 	(wire
 		(pts
+			(xy 40.64 109.22) (xy 40.64 107.95)
+		)
+		(stroke
+			(width 0)
+			(type default)
+		)
+	)
+	(wire
+		(pts
 			(xy 213.36 48.26) (xy 214.63 48.26)
 		)
@@
 	(symbol
 		(lib_id "power:GNDA")
+		(at 40.64 109.22 0)
+		(unit 1)
+		(body_style 1)
+		(exclude_from_sim no)
+		(in_bom yes)
+		(on_board yes)
+		(in_pos_files yes)
+		(dnp no)
+		(fields_autoplaced yes)
+		(property "Reference" "#PWR092"
+			(at 40.64 115.57 0)
+			(hide yes)
+			(show_name no)
+			(do_not_autoplace no)
+			(effects
+				(font
+					(size 1.27 1.27)
+				)
+			)
+		)
+		(property "Value" "GNDA"
+			(at 40.64 114.3 0)
+			(show_name no)
+			(do_not_autoplace no)
+			(effects
+				(font
+					(size 1.27 1.27)
+				)
+			)
+		)
+		(property "Footprint" ""
+			(at 40.64 109.22 0)
+			(hide yes)
+			(show_name no)
+			(do_not_autoplace no)
+			(effects
+				(font
+					(size 1.27 1.27)
+				)
+			)
+		)
+		(property "Datasheet" ""
+			(at 40.64 109.22 0)
+			(hide yes)
+			(show_name no)
+			(do_not_autoplace no)
+			(effects
+				(font
+					(size 1.27 1.27)
+				)
+			)
+		)
+		(property "Description" "Power symbol creates a global label with name \"GNDA\" , analog ground"
+			(at 40.64 109.22 0)
+			(hide yes)
+			(show_name no)
+			(do_not_autoplace no)
+			(effects
+				(font
+					(size 1.27 1.27)
+				)
+			)
+		)
+		(pin "1"
+		)
+		(instances
+			(project "Antenna-Array-Switch-PCB"
+				(path "/53a2d682-f221-4d2b-9002-0fe959bb1f68/43ba60ef-378a-41d1-af5a-6e648ed87248"
+					(reference "#PWR092")
+					(unit 1)
+				)
+			)
+		)
+	)
+	(symbol
+		(lib_id "power:GNDA")
 		(at 158.75 73.66 0)
 		(unit 1)
@@
 	)
 	(symbol
-		(lib_id "power:GNDD")
+		(lib_id "Device:RFShield_OnePiece")
+		(at 40.64 97.79 0)
+		(unit 1)
+		(body_style 1)
+		(exclude_from_sim no)
+		(in_bom yes)
+		(on_board yes)
+		(in_pos_files yes)
+		(dnp no)
+		(fields_autoplaced yes)
+		(property "Reference" "J12"
+			(at 57.15 96.5199 0)
+			(show_name no)
+			(do_not_autoplace no)
+			(effects
+				(font
+					(size 1.27 1.27)
+				)
+				(justify left)
+			)
+		)
+		(property "Value" "RFShield_OnePiece"
+			(at 57.15 99.0599 0)
+			(show_name no)
+			(do_not_autoplace no)
+			(effects
+				(font
+					(size 1.27 1.27)
+				)
+				(justify left)
+			)
+		)
+		(property "Footprint" "RF_Shielding:Wuerth_36103305_30x30mm"
+			(at 40.64 100.33 0)
+			(hide yes)
+			(show_name no)
+			(do_not_autoplace no)
+			(effects
+				(font
+					(size 1.27 1.27)
+				)
+			)
+		)
+		(property "Datasheet" ""
+			(at 40.64 100.33 0)
+			(hide yes)
+			(show_name no)
+			(do_not_autoplace no)
+			(effects
+				(font
+					(size 1.27 1.27)
+				)
+			)
+		)
+		(property "Description" "One-piece EMI RF shielding cabinet"
+			(at 40.64 97.79 0)
+			(hide yes)
+			(show_name no)
+			(do_not_autoplace no)
+			(effects
+				(font
+					(size 1.27 1.27)
+				)
+			)
+		)
+		(pin "1"
+		)
+		(instances
+			(project "Antenna-Array-Switch-PCB"
+				(path "/53a2d682-f221-4d2b-9002-0fe959bb1f68/43ba60ef-378a-41d1-af5a-6e648ed87248"
+					(reference "J12")
+					(unit 1)
+				)
+			)
+		)
+	)
+	(symbol
+		(lib_id "power:GNDA")
 		(at 144.78 157.48 0)
 		(mirror y)
@@
 		(dnp no)
 		(fields_autoplaced yes)
-		(property "Reference" "#PWR043"
+		(property "Reference" "#PWR43"
 			(at 144.78 163.83 0)
 			(hide yes)
@@
 			)
 		)
-		(property "Value" "GNDD"
-			(at 144.78 161.29 0)
+		(property "Value" "GNDA"
+			(at 144.78 162.56 0)
 			(show_name no)
 			(do_not_autoplace no)
@@
 			)
 		)
-		(property "Description" "Power symbol creates a global label with name \"GNDD\" , digital ground"
+		(property "Description" "Power symbol creates a global label with name \"GNDA\" , analog ground"
 			(at 144.78 157.48 0)
 			(hide yes)
@@
 			(project "Antenna-Array-Switch-PCB"
 				(path "/53a2d682-f221-4d2b-9002-0fe959bb1f68/43ba60ef-378a-41d1-af5a-6e648ed87248"
-					(reference "#PWR043")
+					(reference "#PWR43")
 					(unit 1)
 				)
@@
 	)
 	(symbol
-		(lib_id "power:GNDD")
+		(lib_id "power:GNDA")
 		(at 54.61 46.99 270)
 		(unit 1)
@@
 		(dnp no)
 		(fields_autoplaced yes)
-		(property "Reference" "#PWR037"
+		(property "Reference" "#PWR37"
 			(at 48.26 46.99 0)
 			(hide yes)
@@
 			)
 		)
-		(property "Value" "GNDD"
+		(property "Value" "GNDA"
 			(at 50.8 46.9899 90)
 			(show_name no)
@@
 			)
 		)
-		(property "Description" "Power symbol creates a global label with name \"GNDD\" , digital ground"
+		(property "Description" "Power symbol creates a global label with name \"GNDA\" , analog ground"
 			(at 54.61 46.99 0)
 			(hide yes)
@@
 			(project "Antenna-Array-Switch-PCB"
 				(path "/53a2d682-f221-4d2b-9002-0fe959bb1f68/43ba60ef-378a-41d1-af5a-6e648ed87248"
-					(reference "#PWR037")
+					(reference "#PWR37")
 					(unit 1)
 				)
@@
 	)
 	(symbol
-		(lib_id "power:GNDD")
+		(lib_id "power:GNDA")
 		(at 240.03 158.75 0)
 		(unit 1)
@@
 		(dnp no)
 		(fields_autoplaced yes)
-		(property "Reference" "#PWR036"
+		(property "Reference" "#PWR36"
 			(at 240.03 165.1 0)
 			(hide yes)
@@
 			)
 		)
-		(property "Value" "GNDD"
-			(at 240.03 162.56 0)
+		(property "Value" "GNDA"
+			(at 240.03 163.83 0)
 			(show_name no)
 			(do_not_autoplace no)
@@
 			)
 		)
-		(property "Description" "Power symbol creates a global label with name \"GNDD\" , digital ground"
+		(property "Description" "Power symbol creates a global label with name \"GNDA\" , analog ground"
 			(at 240.03 158.75 0)
 			(hide yes)
@@
 			(project "Antenna-Array-Switch-PCB"
 				(path "/53a2d682-f221-4d2b-9002-0fe959bb1f68/43ba60ef-378a-41d1-af5a-6e648ed87248"
-					(reference "#PWR036")
+					(reference "#PWR36")
 					(unit 1)
 				)
@@
 	)
 	(symbol
-		(lib_id "power:GNDD")
+		(lib_id "power:GNDA")
 		(at 99.06 153.67 0)
 		(unit 1)
@@
 		(dnp no)
 		(fields_autoplaced yes)
-		(property "Reference" "#PWR041"
+		(property "Reference" "#PWR41"
 			(at 99.06 160.02 0)
 			(hide yes)
@@
 			)
 		)
-		(property "Value" "GNDD"
-			(at 99.06 157.48 0)
+		(property "Value" "GNDA"
+			(at 99.06 158.75 0)
 			(show_name no)
 			(do_not_autoplace no)
@@
 			)
 		)
-		(property "Description" "Power symbol creates a global label with name \"GNDD\" , digital ground"
+		(property "Description" "Power symbol creates a global label with name \"GNDA\" , analog ground"
 			(at 99.06 153.67 0)
 			(hide yes)
@@
 			(project "Antenna-Array-Switch-PCB"
 				(path "/53a2d682-f221-4d2b-9002-0fe959bb1f68/43ba60ef-378a-41d1-af5a-6e648ed87248"
-					(reference "#PWR041")
+					(reference "#PWR41")
+					(unit 1)
+				)
+			)
+		)
+	)
+	(symbol
+		(lib_id "power:GNDA")
+		(at 135.89 157.48 0)
+		(unit 1)
+		(body_style 1)
+		(exclude_from_sim no)
+		(in_bom yes)
+		(on_board yes)
+		(in_pos_files yes)
+		(dnp no)
+		(fields_autoplaced yes)
+		(property "Reference" "#PWR052"
+			(at 135.89 163.83 0)
+			(hide yes)
+			(show_name no)
+			(do_not_autoplace no)
+			(effects
+				(font
+					(size 1.27 1.27)
+				)
+			)
+		)
+		(property "Value" "GNDA"
+			(at 135.89 162.56 0)
+			(show_name no)
+			(do_not_autoplace no)
+			(effects
+				(font
+					(size 1.27 1.27)
+				)
+			)
+		)
+		(property "Footprint" ""
+			(at 135.89 157.48 0)
+			(hide yes)
+			(show_name no)
+			(do_not_autoplace no)
+			(effects
+				(font
+					(size 1.27 1.27)
+				)
+			)
+		)
+		(property "Datasheet" ""
+			(at 135.89 157.48 0)
+			(hide yes)
+			(show_name no)
+			(do_not_autoplace no)
+			(effects
+				(font
+					(size 1.27 1.27)
+				)
+			)
+		)
+		(property "Description" "Power symbol creates a global label with name \"GNDA\" , analog ground"
+			(at 135.89 157.48 0)
+			(hide yes)
+			(show_name no)
+			(do_not_autoplace no)
+			(effects
+				(font
+					(size 1.27 1.27)
+				)
+			)
+		)
+		(pin "1"
+		)
+		(instances
+			(project "Antenna-Array-Switch-PCB"
+				(path "/53a2d682-f221-4d2b-9002-0fe959bb1f68/43ba60ef-378a-41d1-af5a-6e648ed87248"
+					(reference "#PWR052")
 					(unit 1)
 				)
@@
 					(unit 1)
 				)
-			)
-		)
-	)
-	(symbol
-		(lib_id "power:GNDD")
-		(at 135.89 157.48 0)
-		(unit 1)
-		(body_style 1)
-		(exclude_from_sim no)
-		(in_bom yes)
-		(on_board yes)
-		(in_pos_files yes)
-		(dnp no)
-		(fields_autoplaced yes)
-		(property "Reference" "#PWR042"
-			(at 135.89 163.83 0)
-			(hide yes)
-			(show_name no)
-			(do_not_autoplace no)
-			(effects
-				(font
-					(size 1.27 1.27)
-				)
-			)
-		)
-		(property "Value" "GNDD"
-			(at 135.89 161.29 0)
-			(show_name no)
-			(do_not_autoplace no)
-			(effects
-				(font
-					(size 1.27 1.27)
-				)
-			)
-		)
-		(property "Footprint" ""
-			(at 135.89 157.48 0)
-			(hide yes)
-			(show_name no)
-			(do_not_autoplace no)
-			(effects
-				(font
-					(size 1.27 1.27)
-				)
-			)
-		)
-		(property "Datasheet" ""
-			(at 135.89 157.48 0)
-			(hide yes)
-			(show_name no)
-			(do_not_autoplace no)
-			(effects
-				(font
-					(size 1.27 1.27)
-				)
-			)
-		)
-		(property "Description" "Power symbol creates a global label with name \"GNDD\" , digital ground"
-			(at 135.89 157.48 0)
-			(hide yes)
-			(show_name no)
-			(do_not_autoplace no)
-			(effects
-				(font
-					(size 1.27 1.27)
-				)
-			)
-		)
-		(pin "1"
-		)
-		(instances
-			(project "Antenna-Array-Switch-PCB"
-				(path "/53a2d682-f221-4d2b-9002-0fe959bb1f68/43ba60ef-378a-41d1-af5a-6e648ed87248"
-					(reference "#PWR042")
-					(unit 1)
-				)

Commit message: PCB: Replicate layouts to all LNA chains
Parts:
- renumbered D10 to D201, D7 to D202, D8 to D203, D9 to D204, J12 to J201, R16 to R201, R17 to R202, R18 to R203, R19 to R204, R20 to R205, R21 to R206, R22 to R207, R23 to R208, R24 to R209, R14 to R210, R13 to R211, R15 to R212, SW1 to SW201, SW2 to SW202, U9 to U201
