File: Antenna-Array-Switch-PCB/Antenna-Array-Switch-PCB.kicad_pcb (KiCad board)
At the start: 4 copper layers, 98 x 98 mm, 197 parts, among them J1001 Conn_Coaxial, J101 Conn_SMA, J102 Conn_SMA, J103 Conn_SMA, J104 Conn_Coaxial, J201 RFShield_OnePiece, J301 Conn_Coaxial, J401 Conn_Coaxial, J501 Conn_Coaxial, J601 Conn_Coaxial, J701 Conn_Coaxial, J801 Conn_Coaxial, J901 Conn_Coaxial, SW201 TS-1187A-B-A-B, SW202 TS-1187A-B-A-B, U1001 TPS22917DBV, U1002 PGA-103+, U101 LM1117IMP-3.3, U102 SKY13418-485LF, U201 RP2040-Zero, U301 TPS22917DBV, U302 PGA-103+, U401 TPS22917DBV, U402 PGA-103+, U501 TPS22917DBV, U502 PGA-103+, U601 TPS22917DBV, U602 PGA-103+, U701 TPS22917DBV, U702 PGA-103+, U801 TPS22917DBV, U802 PGA-103+, U901 TPS22917DBV, U902 PGA-103+

Commit message: PCB: Minor review updates - vias, DC block on switch output
Parts:
- added C112: 100pF, Capacitor_SMD:C_0603_1608Metric_Pad1.08x0.95mm_HandSolder, F.Cu at (149.5, 103.4)
- moved J103 0.65 mm to (149.8, 109.4)
Connections:
- U102 pad 13: Net-(J103-In) -> Net-(U102-ANT)
Routing:
- net Net-(J103-In): track 7.58 -> 5.26 mm
- net Net-(U102-ANT): track 0.00 -> 1.26 mm
- net GNDA: vias 1207 -> 1242
Other:
- board text added: "Rev 1 | 2026-10-20"
- board text removed: "Rev 1 | 2026-10-19"
